File: miditwiddle.kicad_pcb (KiCad board)
At the start: 2 copper layers, 98 x 51 mm, 39 parts, among them J1 9V DC In, J2 AVR-ISP, J3 MIDI In, J4 MIDI Out, SW1 Power, SW2 Reset, SW3 Switch, SW4 Button, SW5 Rotary_Enc, U1 MCP1700-5002E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

Commit message: Migrate project to KiCad 6
Parts:
- D2: value 1N914 -> 1N1418
- U1: value MCP1700-5002E -> MCP1702-5002E
Connections:
- net ~Reset renamed ~{Reset}
- J3 pad 1: Net-(J3-Pad1) -> unconnected-(J3-Pad1)
- J3 pad 2: Net-(J3-Pad2) -> unconnected-(J3-Pad2)
- J3 pad 3: Net-(J3-Pad3) -> unconnected-(J3-Pad3)
- J4 pad 1: Net-(J4-Pad1) -> unconnected-(J4-Pad1)
- J4 pad 3: Net-(J4-Pad3) -> unconnected-(J4-Pad3)
- SW1 pad 1: Net-(SW1-Pad1) -> unconnected-(SW1-Pad1)
- SW3 pad 3: Net-(SW3-Pad3) -> unconnected-(SW3-Pad3)
- U2 pad 11: Net-(U2-Pad11) -> unconnected-(U2-Pad11)
- U2 pad 16: Net-(U2-Pad16) -> unconnected-(U2-Pad16)
- U2 pad 9: Net-(U2-Pad9) -> unconnected-(U2-Pad9)
- U3 pad 1: Net-(U3-Pad1) -> unconnected-(U3-Pad1)
- U3 pad 4: Net-(U3-Pad4) -> unconnected-(U3-Pad4)
- U3 pad 7: Net-(U3-Pad7) -> unconnected-(U3-Pad7)
Other:
- net class Default removed
- net class Power removed
